Commit message: first stage of simulator - simple case with rigid model equiped with cameras and imu, model with flexibility/springs in joints not tested enough; launch files to run different environments - with moon gravity and surface as flat or 3D model; trajectory generator node as sandbox for python learning - not functional

File: galago_gazebo_models/urdf/galago_simple/galago_simple.urdf (robot description, URDF)
Before this commit: robot galago_simple, 1 links, 0 joints
Links:
- removed link chassis
- added link body, mass 10.0; collision mesh filename=package://galago_gazebo_models/meshes/galago_simple/galago_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; visual mesh filename=package://galago_gazebo_models/meshes/galago_simple/galago_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
- added link cam_a_link; visual box size=0.1 0.1 0.1
- added link cam_b_link; visual box size=0.1 0.1 0.1
- added link cam_c_link; visual box size=0.1 0.1 0.1
- added link cam_down_link; visual box size=0.1 0.1 0.1
- added link cam_up_link; visual box size=0.1 0.1 0.1
Joints:
- added joint cam_a_joint: type fixed, parent body, child cam_a_link, origin xyz=-0.5 0 0.5 rpy=0 0 3.1416
- added joint cam_b_joint: type fixed, parent body, child cam_b_link, origin xyz=0.25 -0.433 0.5 rpy=0 0 -1.0472
- added joint cam_c_joint: type fixed, parent body, child cam_c_link, origin xyz=0.25 0.433 0.5 rpy=0 0 1.0472
- added joint cam_down_joint: type fixed, parent body, child cam_down_link, origin xyz=0.0 0.0 0.5 rpy=0 1.57 0
- added joint cam_up_joint: type fixed, parent body, child cam_up_link, origin xyz=0.0 0.0 0.5 rpy=0 -1.57 0
